Commit message: Complete Hand_f config

File: src/curobo/content/assets/robot/hand_f/hand_f_before.urdf (robot description, URDF)
Before this commit: robot right_hand_f, 17 links, 16 joints
Links:
- link rh_ffdistal: mass 0.00529857938896386 -> 0.00529857877771826; geometry collision mesh filename=meshes/link1.3.STL; visual mesh filename=meshes/link1.3.STL
- link rh_ffmiddle: mass 0.00324244182122049 -> 0.00324240874433465; geometry collision mesh filename=meshes/link1.2.STL; visual mesh filename=meshes/link1.2.STL
- link rh_ffproximal: mass 0.00677367505247576 -> 0.00677364247310552; geometry collision mesh filename=meshes/link1.1.STL; visual mesh filename=meshes/link1.1.STL
- link rh_lfdistal: mass 0.00529857877771826 -> 0.00529857938896386; geometry collision mesh filename=meshes/link4.3.STL; visual mesh filename=meshes/link4.3.STL
- link rh_lfmiddle: mass 0.00324240874433465 -> 0.00324244182122049; geometry collision mesh filename=meshes/link4.2.STL; visual mesh filename=meshes/link4.2.STL
- link rh_lfproximal: mass 0.00677364247310552 -> 0.00677367505247576; geometry collision mesh filename=meshes/link4.1.STL; visual mesh filename=meshes/link4.1.STL
- link rh_mfdistal: mass 0.0052985823368308 -> 0.00529858100427292; geometry collision mesh filename=meshes/link2.3.STL; visual mesh filename=meshes/link2.3.STL
- link rh_mfmiddle: mass 0.00324244064669766 -> 0.00324240601749207; geometry collision mesh filename=meshes/link2.2.STL; visual mesh filename=meshes/link2.2.STL
- link rh_mfproximal: mass 0.00677364781232352 -> 0.00677364542683526; geometry collision mesh filename=meshes/link2.1.STL; visual mesh filename=meshes/link2.1.STL
- link rh_rfdistal: mass 0.00529858100427292 -> 0.0052985823368308; geometry collision mesh filename=meshes/link3.3.STL; visual mesh filename=meshes/link3.3.STL
- link rh_rfmiddle: mass 0.00324240601749207 -> 0.00324244064669766; geometry collision mesh filename=meshes/link3.2.STL; visual mesh filename=meshes/link3.2.STL
- link rh_rfproximal: mass 0.00677364542683526 -> 0.00677364781232352; geometry collision mesh filename=meshes/link3.1.STL; visual mesh filename=meshes/link3.1.STL
Joints:
- joint rh_FFJ3: origin xyz=0.017201 -0.0099 0.066114 rpy=-3.1416 1.3587 -3.1416 -> xyz=-0.049344 -0.0099 0.056068 rpy=0 1.1345 0
- joint rh_LFJ3: origin xyz=-0.049344 -0.0099 0.056068 rpy=0 1.1345 0 -> xyz=0.017201 -0.0099 0.066114 rpy=-3.1416 1.3587 -3.1416
- joint rh_MFJ3: origin xyz=-0.005458 -0.0099 0.067348 rpy=-3.1416 1.5681 -3.1416 -> xyz=-0.027527 -0.0099 0.064462 rpy=0 1.3989 0
- joint rh_RFJ3: origin xyz=-0.027527 -0.0099 0.064462 rpy=0 1.3989 0 -> xyz=-0.005458 -0.0099 0.067348 rpy=-3.1416 1.5681 -3.1416

File: src/curobo/content/assets/robot/hand_f/hand_f_before2.urdf (robot description, URDF)
Before this commit: robot right_hand_f, 17 links, 16 joints
Links:
- link rh_ffdistal: mass 0.00529857938896386 -> 0.00529857877771826; geometry collision mesh filename=meshes/link1.3.STL; visual mesh filename=meshes/link1.3.STL
- link rh_ffmiddle: mass 0.00324244182122049 -> 0.00324240874433465; geometry collision mesh filename=meshes/link1.2.STL; visual mesh filename=meshes/link1.2.STL
- link rh_ffproximal: mass 0.00677367505247576 -> 0.00677364247310552; geometry collision mesh filename=meshes/link1.1.STL; visual mesh filename=meshes/link1.1.STL
- link rh_lfdistal: mass 0.00529857877771826 -> 0.00529857938896386; geometry collision mesh filename=meshes/link4.3.STL; visual mesh filename=meshes/link4.3.STL
- link rh_lfmiddle: mass 0.00324240874433465 -> 0.00324244182122049; geometry collision mesh filename=meshes/link4.2.STL; visual mesh filename=meshes/link4.2.STL
- link rh_lfproximal: mass 0.00677364247310552 -> 0.00677367505247576; geometry collision mesh filename=meshes/link4.1.STL; visual mesh filename=meshes/link4.1.STL
- link rh_mfdistal: mass 0.0052985823368308 -> 0.00529858100427292; geometry collision mesh filename=meshes/link2.3.STL; visual mesh filename=meshes/link2.3.STL
- link rh_mfmiddle: mass 0.00324244064669766 -> 0.00324240601749207; geometry collision mesh filename=meshes/link2.2.STL; visual mesh filename=meshes/link2.2.STL
- link rh_mfproximal: mass 0.00677364781232352 -> 0.00677364542683526; geometry collision mesh filename=meshes/link2.1.STL; visual mesh filename=meshes/link2.1.STL
- link rh_rfdistal: mass 0.00529858100427292 -> 0.0052985823368308; geometry collision mesh filename=meshes/link3.3.STL; visual mesh filename=meshes/link3.3.STL
- link rh_rfmiddle: mass 0.00324240601749207 -> 0.00324244064669766; geometry collision mesh filename=meshes/link3.2.STL; visual mesh filename=meshes/link3.2.STL
- link rh_rfproximal: mass 0.00677364542683526 -> 0.00677364781232352; geometry collision mesh filename=meshes/link3.1.STL; visual mesh filename=meshes/link3.1.STL
Joints:
- joint rh_FFJ1: limit lower=-1.30899694 upper=1.30899694 effort=1 velocity=1 -> lower=-1.570796326790 upper=0.000000000000 effort=100 velocity=100
- joint rh_FFJ2: limit lower=-1.30899694 upper=1.30899694 effort=1 velocity=1 -> lower=-1.570796326790 upper=0.000000000000 effort=100 velocity=100
- joint rh_FFJ3: limit lower=-1.30899694 upper=1.30899694 effort=1 velocity=1 -> lower=-1.570796326790 upper=0.261799387799 effort=100 velocity=100; origin xyz=0.017201 -0.0099 0.066114 rpy=-3.1416 1.3587 -3.1416 -> xyz=-0.049344 -0.0099 0.056068 rpy=0 1.1345 0
- joint rh_LFJ1: limit lower=-1.30899694 upper=1.30899694 effort=1 velocity=1 -> lower=-1.570796326790 upper=0.000000000000 effort=100 velocity=100
- joint rh_LFJ2: limit lower=-1.30899694 upper=1.30899694 effort=1 velocity=1 -> lower=-1.570796326790 upper=0.000000000000 effort=100 velocity=100
- joint rh_LFJ3: limit lower=-1.30899694 upper=1.30899694 effort=1 velocity=1 -> lower=-1.570796326790 upper=0.261799387799 effort=100 velocity=100; origin xyz=-0.049344 -0.0099 0.056068 rpy=0 1.1345 0 -> xyz=0.017201 -0.0099 0.066114 rpy=-3.1416 1.3587 -3.1416
- joint rh_MFJ1: limit lower=-1.30899694 upper=1.30899694 effort=1 velocity=1 -> lower=-1.570796326790 upper=0.000000000000 effort=100 velocity=100
- joint rh_MFJ2: axis 0 0 -1 -> 0 0 1; limit lower=-1.30899694 upper=1.30899694 effort=1 velocity=1 -> lower=-1.570796326790 upper=0.000000000000 effort=100 velocity=100
- joint rh_MFJ3: limit lower=-1.30899694 upper=1.30899694 effort=1 velocity=1 -> lower=-1.570796326790 upper=0.261799387799 effort=100 velocity=100; origin xyz=-0.005458 -0.0099 0.067348 rpy=-3.1416 1.5681 -3.1416 -> xyz=-0.027527 -0.0099 0.064462 rpy=0 1.3989 0
- joint rh_RFJ1: limit lower=-1.30899694 upper=1.30899694 effort=1 velocity=1 -> lower=-1.570796326790 upper=0.000000000000 effort=100 velocity=100
- joint rh_RFJ2: limit lower=-1.30899694 upper=1.30899694 effort=1 velocity=1 -> lower=-1.570796326790 upper=0.000000000000 effort=100 velocity=100
- joint rh_RFJ3: limit lower=-1.30899694 upper=1.30899694 effort=1 velocity=1 -> lower=-1.570796326790 upper=0.261799387799 effort=100 velocity=100; origin xyz=-0.027527 -0.0099 0.064462 rpy=0 1.3989 0 -> xyz=-0.005458 -0.0099 0.067348 rpy=-3.1416 1.5681 -3.1416
- joint rh_THJ1: limit lower=-1.30899694 upper=1.30899694 effort=1 velocity=1 -> lower=-1.570796326790 upper=0.261799387799 effort=100 velocity=100
- joint rh_THJ2: limit lower=-1.30899694 upper=1.30899694 effort=1 velocity=1 -> lower=-0.698131700798 upper=0.698131700798 effort=100 velocity=100
- joint rh_THJ3: limit lower=-1.30899694 upper=1.30899694 effort=1 velocity=1 -> lower=-0.209439510239 upper=0.209439510239 effort=100 velocity=100
- joint rh_THJ4: limit lower=-1.30899694 upper=1.30899694 effort=1 velocity=1 -> lower=-1.221730476400 upper=0.000000000000 effort=100 velocity=100
